File: project/ecad/carte-principale/carte principale.kicad_pcb (KiCad board)
At the start: 4 copper layers, 99 x 163 mm, 152 parts, among them J1 ecran tft, J10 Conn_01x04, J11 Conn_01x04, J4 Conn_01x04, J5 LIDAR, J6 BAU, J7 Conn_01x04, J8 Conn_01x04, J9 Conn_01x04, K2 G2RL-1-E, U1 TSR1-2433E, U10 TMC2209, U11 PCA9685PW, U2 TSR1-2450E, U3 PCA9685PW, U4 ESP32-S3-DevKitC, U5 TMC2209, U6 TMC2209, U7 TMC2209, U8 TMC2209, U9 TMC2209

Commit message: ajout dossier pcb
Parts:
- removed C10, C8: 10u, Capacitor_THT:CP_Radial_D10.0mm_P5.00mm
- removed C20, C23: 10u, Capacitor_SMD:C_1206_3216Metric_Pad1.33x1.80mm_HandSolder
- removed J11, J9: Conn_01x04, Connector_Molex:Molex_KK-254_AE-6410-04A_1x04_P2.54mm_Vertical
- removed JP17, JP18, JP20, JP21: SolderJumper_3_Open, Jumper:SolderJumper-3_P1.3mm_Open_RoundedPad1.0x1.5mm
- removed U10, U7: TMC2209, Library:MODULE_TMC2209_SILENTSTEPSTICK
- added Button2: Conn_01x02, Connector_Molex:Molex_KK-254_AE-6410-02A_1x02_P2.54mm_Vertical, F.Cu at (92.0, 83.0)
- added C53: 10u, Capacitor_SMD:C_1206_3216Metric_Pad1.33x1.80mm_HandSolder, F.Cu at (124.5, 156.0)
- added G***: LOGO, LOGO, F.Cu at (150.0, 169.0)
- added G***: LOGO, LOGO, F.Cu at (198.2, 113.0)
- added G***: LOGO, LOGO, F.Cu at (114.4, 131.8)
- added G***: LOGO, LOGO, F.Cu at (65.6, 156.8)
- added G***: LOGO, LOGO, F.Cu at (62.4, 105.1)
- added ICM1: PCF8574T, Package_SO:SOIC-16W_7.5x10.3mm_P1.27mm, F.Cu at (102.7, 118.5)
- added JP12: SolderJumper_2_Open, Jumper:SolderJumper-2_P1.3mm_Open_RoundedPad1.0x1.5mm, F.Cu at (100.7, 110.5)
- added JP13: SolderJumper_2_Open, Jumper:SolderJumper-2_P1.3mm_Open_RoundedPad1.0x1.5mm, F.Cu at (104.7, 110.5)
- added R35: 4.7k, Resistor_SMD:R_1206_3216Metric_Pad1.30x1.75mm_HandSolder, F.Cu at (100.7, 105.8)
- added R36: 4.7k, Resistor_SMD:R_1206_3216Metric_Pad1.30x1.75mm_HandSolder, F.Cu at (104.7, 105.8)
- added R37: 4.7k, Resistor_SMD:R_1206_3216Metric_Pad1.30x1.75mm_HandSolder, F.Cu at (105.7, 125.5)
- added switch3: Conn_01x02, Connector_Molex:Molex_KK-254_AE-6410-02A_1x02_P2.54mm_Vertical, F.Cu at (92.0, 110.9)
- added switch4: Conn_01x02, Connector_Molex:Molex_KK-254_AE-6410-02A_1x02_P2.54mm_Vertical, F.Cu at (92.0, 103.9)
- added switch5: Conn_01x02, Connector_Molex:Molex_KK-254_AE-6410-02A_1x02_P2.54mm_Vertical, F.Cu at (92.0, 97.0)
- C5, C6, C7, C9: value 10u -> 100u
- moved C16 114.0 mm to (150.0, 70.0), turned to 90 degrees
- moved C21 113.2 mm to (105.5, 153.0), turned to -90 degrees
- moved switch2 93.6 mm to (92.0, 117.9), turned to 90 degrees
- moved switch1 78.6 mm to (92.0, 124.9), turned to 90 degrees
- moved Button1 50.8 mm to (92.0, 90.0), turned to 90 degrees
- moved C19 43.8 mm to (105.5, 174.0), turned to -90 degrees
- moved Tirette1 43.8 mm to (92.0, 76.0), turned to 90 degrees
- moved JP1 43.7 mm to (95.5, 163.0), turned to 180 degrees
- moved JP2 43.5 mm to (95.5, 166.0), turned to 180 degrees
- moved U5 43.5 mm to (95.5, 165.0), turned to 180 degrees
- moved JP6 42.4 mm to (134.5, 146.0), turned to 0 degrees
- moved U9 41.4 mm to (134.5, 144.0), turned to 0 degrees
- moved C6 40.3 mm to (132.1, 174.0)
- moved JP19 39.7 mm to (134.5, 143.0), turned to 0 degrees
- moved C5 38.8 mm to (97.9, 156.0), turned to 180 degrees
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- renumbered BAU1 to BAU, Batt1 to Batt
Connections:
- Button1 pad 1: /bu -> /bu 1
- Tirette1 pad 2: GND -> unconnected-(Tirette1-Pin_2-Pad2)
- U4 pad 10: /RX -> SDA
- U4 pad 11: /TX -> /pwm
- U4 pad 12: SDA -> /RX
- U4 pad 14: SCL -> unconnected-(U4-GPIO46-Pad14)
- U4 pad 15: /oe -> /TX
- U4 pad 16: /sck -> /sdo
- U4 pad 17: /sdi -> /sck
- U4 pad 18: /dc -> /sdi
- U4 pad 19: /cs -> /dc
- U4 pad 20: /sw2 -> /cs
- U4 pad 27: DIR 3 -> /tir
- U4 pad 28: STEP 5 -> /bu 2
- U4 pad 29: DIR 5 -> /bu 1
- U4 pad 32: STEP 4 -> unconnected-(U4-GPIO35-Pad32)
- U4 pad 33: DIR 4 -> unconnected-(U4-GPIO36-Pad33)
- U4 pad 34: STEP 6 -> unconnected-(U4-GPIO37-Pad34)
- U4 pad 35: DIR 6 -> unconnected-(U4-GPIO38-Pad35)
- U4 pad 36: /tir -> STEP 3
- U4 pad 37: /bu -> DIR 3
- U4 pad 38: /pwm -> STEP 1
- U4 pad 39: /sw1 -> DIR 1
- U4 pad 4: STEP 1 -> STEP 2
- U4 pad 40: Net-(U10-~{EN}) -> En5VP
- U4 pad 41: En5VP -> /En driver
- U4 pad 5: DIR 1 -> DIR 2
- U4 pad 6: STEP 2 -> STEP 4
- U4 pad 7: /sdo -> DIR 4
- U4 pad 8: DIR 2 -> /oe
- U4 pad 9: STEP 3 -> SCL
- U5 pad 16: Net-(U10-~{EN}) -> /En driver
- U6 pad 16: Net-(U10-~{EN}) -> /En driver
- U8 pad 10: STEP 4 -> STEP 3
- U8 pad 16: Net-(U10-~{EN}) -> /En driver
- U8 pad 9: DIR 4 -> DIR 3
- U9 pad 10: STEP 5 -> STEP 4
- U9 pad 16: Net-(U10-~{EN}) -> /En driver
- U9 pad 9: DIR 5 -> DIR 4
Routing:
- net Net-(U10-~{EN}): track 202.5 -> 0.00 mm
- net /En driver: track 0.00 -> 151.9 mm
- net STEP 6: track 131.4 -> 0.00 mm
- net DIR 6: track 130.4 -> 0.00 mm
- net GND: track 179.7 -> 67.5 mm, vias 56 -> 196
- net STEP 5: track 106.1 -> 0.00 mm
- net DIR 5: track 105.5 -> 0.00 mm
- net +5VP: track 583.8 -> 511.7 mm
- net +24V: track 258.4 -> 214.1 mm, vias 74 -> 59
- net SDA: track 83.7 -> 126.3 mm, vias 2 -> 3
- net SCL: track 86.0 -> 125.6 mm, vias 2 -> 3
- net STEP 4: track 116.2 -> 78.7 mm
- net DIR 4: track 115.7 -> 79.0 mm
- net /bu: track 32.4 -> 0.00 mm
- net /sw5: track 0.00 -> 30.9 mm
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- added copper zone on F.Cu, net GND
Other:
- board size 99 x 163 mm -> 99 x 146 mm
- board text added: "100u"
- board text added: "10k"
- board text added: "10u"
- board text added: "1k"
- board text added: "220u"
- board text added: "24V"
- board text added: "3V3"
- board text added: "4.7k"
- board text added: "5VL"
- board text added: "5VP"
- board text added: "Batt"
- board text added: "G2RL-1-E"
- board text added: "Lapeyronnie Paul co-président UniMakers 17/10/2026"
- board text added: "Lidar"
- board text added: "Moteur"
- board text added: "PCA9685PW"
- board text added: "TMC2209"
- board text added: "ecran tft"
