File: project/ecad/carte-principale/carte principale.kicad_sch (KiCad schematic)
At the start: 152 parts, among them J1 ecran tft, J10 Conn_01x04, J11 Conn_01x04, J4 Conn_01x04, J5 LIDAR, J6 BAU, J7 Conn_01x04, J8 Conn_01x04, J9 Conn_01x04, K2 G2RL-1-E, U1 TSR1-2433E, U10 TMC2209, U11 PCA9685PW, U2 TSR1-2450E, U3 PCA9685PW, U4 ESP32-S3-DevKitC, U5 TMC2209, U6 TMC2209, U7 TMC2209, U8 TMC2209, U9 TMC2209

Commit message: ajout dossier pcb
Parts:
- removed C10, C8: 10u, Capacitor_THT:CP_Radial_D10.0mm_P5.00mm, symbol Device:C_Polarized_Small
- removed C20, C23: 10u, Capacitor_SMD:C_1206_3216Metric_Pad1.33x1.80mm_HandSolder, symbol Device:C_Small
- removed J11, J9: Conn_01x04, Connector_Molex:Molex_KK-254_AE-6410-04A_1x04_P2.54mm_Vertical, symbol Connector_Generic:Conn_01x04
- removed JP17, JP18, JP20, JP21: SolderJumper_3_Open, Jumper:SolderJumper-3_P1.3mm_Open_RoundedPad1.0x1.5mm, symbol Jumper:SolderJumper_3_Open
- removed U10, U7: TMC2209, Library:MODULE_TMC2209_SILENTSTEPSTICK, symbol TMC2209_SILENTSTEPSTICK:TMC2209_SILENTSTEPSTICK
- added Button2, switch3, switch4, switch5: Conn_01x02, Connector_Molex:Molex_KK-254_AE-6410-02A_1x02_P2.54mm_Vertical, symbol Connector_Generic:Conn_01x02
- added C53: 10u, Capacitor_SMD:C_1206_3216Metric_Pad1.33x1.80mm_HandSolder, symbol Device:C_Small
- added ICM1: PCF8574T, Package_SO:SOIC-16W_7.5x10.3mm_P1.27mm, symbol Interface_Expansion:PCF8574T
- added JP12, JP13: SolderJumper_2_Open, Jumper:SolderJumper-2_P1.3mm_Open_RoundedPad1.0x1.5mm, symbol Jumper:SolderJumper_2_Open
- added R35, R36, R37: 4.7k, Resistor_SMD:R_1206_3216Metric_Pad1.30x1.75mm_HandSolder, symbol Device:R_Small
- C5, C6, C7, C9: value 10u -> 100u
Connections:
- net +3V3: now also C53.1, ICM1.16 (VDD), JP12.1 (A), JP13.1 (A), R37.1
- net DIR 1: now also U4.39 (GPIO42/MTMS); no longer U4.5 (GPIO5/ADC1_CH4)
- net DIR 2: now also U4.5 (GPIO5/ADC1_CH4); no longer U4.8 (GPIO15/ADC2_CH4/32K_P)
- net DIR 3: now also U4.37 (GPIO40/MTDO), U8.9 (DIR); no longer U4.27 (GPIO21)
- net DIR 4: now also U4.7 (GPIO7/ADC1_CH6), U9.9 (DIR); no longer U4.33 (GPIO36), U8.9 (DIR)
- net En5VP: now also U4.40 (GPIO2/ADC1_CH1); no longer U4.41 (GPIO1/ADC1_CH0)
- net GND: now also Button2.2 (Pin_2), C53.2, ICM1.3 (A2), ICM1.8 (GND), R35.2, R36.2, switch3.2 (Pin_2), switch4.2 (Pin_2), switch5.2 (Pin_2); no longer Tirette1.2 (Pin_2)
- net RX: now also U4.12 (GPIO8/ADC1_CH7); no longer U4.10 (GPIO17/ADC2_CH6)
- net SCL: now also U4.9 (GPIO16/ADC2_CH5/32K_N), ICM1.14 (SCL); no longer U4.14 (GPIO46)
- net SDA: now also U4.10 (GPIO17/ADC2_CH6), ICM1.15 (SDA); no longer U4.12 (GPIO8/ADC1_CH7)
- net STEP 1: now also U4.38 (GPIO41/MTDI); no longer U4.4 (GPIO4/ADC1_CH3)
- net STEP 2: now also U4.4 (GPIO4/ADC1_CH3); no longer U4.6 (GPIO6/ADC1_CH5)
- net STEP 3: now also U4.36 (GPIO39/MTCK), U8.10 (STEP); no longer U4.9 (GPIO16/ADC2_CH5/32K_N)
- net STEP 4: now also U4.6 (GPIO6/ADC1_CH5), U9.10 (STEP); no longer U4.32 (GPIO35), U8.10 (STEP)
- net TX: now also U4.15 (GPIO9/ADC1_CH8); no longer U4.11 (GPIO18/ADC2_CH7)
- net cs: now also U4.20 (GPIO14/ADC2_CH3); no longer U4.19 (GPIO13/ADC2_CH2)
- net dc: now also U4.19 (GPIO13/ADC2_CH2); no longer U4.18 (GPIO12/ADC2_CH1)
- net oe: now also U4.8 (GPIO15/ADC2_CH4/32K_P); no longer U4.15 (GPIO9/ADC1_CH8)
- net pwm: now also U4.11 (GPIO18/ADC2_CH7); no longer U4.38 (GPIO41/MTDI)
- net sck: now also U4.17 (GPIO11/ADC2_CH0); no longer U4.16 (GPIO10/ADC1_CH9)
- net sdi: now also U4.18 (GPIO12/ADC2_CH1); no longer U4.17 (GPIO11/ADC2_CH0)
- net sdo: now also U4.16 (GPIO10/ADC1_CH9); no longer U4.7 (GPIO7/ADC1_CH6)
- net sw1: now also ICM1.12 (P7); no longer U4.39 (GPIO42/MTMS)
- net sw2: now also ICM1.11 (P6); no longer U4.20 (GPIO14/ADC2_CH3)
- net tir: now also U4.27 (GPIO21); no longer U4.36 (GPIO39/MTCK)
- net En driver: now reaches U5.16 (~{EN}), U6.16 (~{EN}), U8.16 (~{EN}), U9.16 (~{EN})
- net En driver: now also U4.41 (GPIO1/ADC1_CH0); no longer U4.40 (GPIO2/ADC1_CH1)
- net DIR 5 renamed bu 1
- net bu 1: now also Button1.1 (Pin_1); no longer U9.9 (DIR)
- net DIR 6: no longer names the net of U4.35 (GPIO38)
- net STEP 5 renamed bu 2
- net bu 2: now also Button2.1 (Pin_1); no longer U9.10 (STEP)
- net STEP 6: no longer names the net of U4.34 (GPIO37)
- removed net bu: Button1.1 (Pin_1), U4.37 (GPIO40/MTDO)
- new net: ICM1.2 (A1), JP13.2 (B), R36.1
- new net: ICM1.1 (A0), JP12.2 (B), R35.1
- new net: ICM1.13 (~{INT}), R37.2
- new net sw3: ICM1.10 (P5), switch3.1 (Pin_1)
- new net sw4: ICM1.9 (P4), switch4.1 (Pin_1)
- new net sw5: ICM1.7 (P3), switch5.1 (Pin_1)
- no-connect marks 41 -> 39
Other:
- moved on the sheet: BAU1, Batt1, C12, C13, C14, C16, C17, C24, C25, C26, C27, C28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
